Commit message: first major update, adding teleoperation for a climbing robot

File: sim/pybullet/urdf_scalar_6DoF/urdf/wall_camera_manyholds.urdf (robot description, URDF)
Before this commit: robot wall_with_hold, 9 links, 8 joints
Links:
- link hold5: geometry collision box size=0.05 0.07 0.0; visual box size=0.05 0.07 0.0
Joints:
- joint wall_hold_joint: origin xyz=-0.12 0.3 0.05 rpy=3.14 0 0.0 -> xyz=-0.12 0.32 0.07 rpy=3.14 0 0.0
- joint wall_hold_joint2: origin xyz=-0.12 0.3 0.05 rpy=3.14 0 0.0 -> xyz=0.12 0.42 0.07 rpy=3.14 0 0.0
- joint wall_hold_joint3: origin xyz=-0.12 0.3 0.05 rpy=3.14 0 0.0 -> xyz=0.12 -0.32 0.07 rpy=3.14 0 0.0
- joint wall_hold_joint4: origin xyz=-0.12 0.3 0.05 rpy=3.14 0 0.0 -> xyz=-0.12 -0.32 0.07 rpy=3.14 0 0.0
- joint wall_hold_joint5: origin xyz=-0.22 0.3 0.05 rpy=3.14 0 0.0 -> xyz=-0.12 0.5 0.07 rpy=3.14 0 0.0
