Commit message: Replaced the old parallel jaw gripper to the GOAT gripper.

File: sim/pybullet/urdf_scalar_6DoF/urdf/SCALAR_6DoF_gripper_test.urdf (robot description, URDF)
Before this commit: robot SCALAR_6DoF, 70 links, 69 joints
Links:
- removed link finger_left0
- removed link finger_left1
- removed link finger_left2
- removed link finger_left3
- removed link finger_right0
- removed link finger_right1
- removed link finger_right2
- removed link finger_right3
- removed link gripper_left0
- removed link gripper_left1
- removed link gripper_left2
- removed link gripper_left3
- removed link gripper_right0
- removed link gripper_right1
- removed link gripper_right2
- removed link gripper_right3
- added link left_finger, mass 0.024207; collision mesh filename=left_finger.STL; visual mesh filename=left_finger.STL
- added link left_finger1, mass 0.024207; collision mesh filename=left_finger.STL; visual mesh filename=left_finger.STL
- added link left_finger2, mass 0.024207; collision mesh filename=left_finger.STL; visual mesh filename=left_finger.STL
- added link left_finger3, mass 0.024207; collision mesh filename=left_finger.STL; visual mesh filename=left_finger.STL
- added link right_finger, mass 0.024207; collision mesh filename=right_finger.STL; visual mesh filename=right_finger.STL
- added link right_finger1, mass 0.024207; collision mesh filename=right_finger.STL; visual mesh filename=right_finger.STL
- added link right_finger2, mass 0.024207; collision mesh filename=right_finger.STL; visual mesh filename=right_finger.STL
- added link right_finger3, mass 0.024207; collision mesh filename=right_finger.STL; visual mesh filename=right_finger.STL
- link base_link_gripper0: mass 1.2 -> 0.067952; geometry collision mesh filename=base_link.STL; visual mesh filename=base_link.STL
- link base_link_gripper1: mass 1.2 -> 0.067952; geometry collision mesh filename=base_link.STL; visual mesh filename=base_link.STL
- link base_link_gripper2: mass 1.2 -> 0.067952; geometry collision mesh filename=base_link.STL; visual mesh filename=base_link.STL
- link base_link_gripper3: mass 1.2 -> 0.067952; geometry collision mesh filename=base_link.STL; visual mesh filename=base_link.STL
Joints:
- removed joint guide_joint_finger_left0
- removed joint guide_joint_finger_left1
- removed joint guide_joint_finger_left2
- removed joint guide_joint_finger_left3
- removed joint guide_joint_finger_right0
- removed joint guide_joint_finger_right1
- removed joint guide_joint_finger_right2
- removed joint guide_joint_finger_right3
- joint attachment_joint0: origin xyz=0 0 0.075 rpy=0 0 0 -> xyz=-0.03 0 0.075 rpy=3.14 0 1.57
- joint attachment_joint1: origin xyz=0 0 0.075 rpy=0 0 3.14 -> xyz=0.03 0 0.075 rpy=3.14 0 1.57
- joint attachment_joint2: origin xyz=0 0 0.075 rpy=0 0 3.14 -> xyz=-0.03 0 0.075 rpy=3.14 0 1.57
- joint attachment_joint3: origin xyz=0 0 0.075 rpy=0 0 0 -> xyz=0.03 0 0.075 rpy=3.14 0 1.57
- joint base_joint_gripper_left0: axis 1 0 0 -> 0 1 0; child gripper_left0 -> left_finger; limit lower=-0.055 upper=-0.0027 effort=1.0 velocity=1.0 -> lower=0.01 upper=0.065 effort=0 velocity=0; origin xyz=0 0 0 rpy=0 0 0 -> xyz=0.0080046 -0.005 -0.055798 rpy=1.5708 -1.5708 0
- joint base_joint_gripper_left1: axis 1 0 0 -> 0 1 0; child gripper_left1 -> left_finger1; limit lower=-0.055 upper=-0.0027 effort=1.0 velocity=1.0 -> lower=0.01 upper=0.065 effort=0 velocity=0; origin xyz=0 0 0 rpy=0 0 0 -> xyz=0.0080046 -0.005 -0.055798 rpy=1.5708 -1.5708 0
- joint base_joint_gripper_left2: axis 1 0 0 -> 0 1 0; child gripper_left2 -> left_finger2; limit lower=-0.055 upper=-0.0027 effort=1.0 velocity=1.0 -> lower=0.01 upper=0.065 effort=0 velocity=0; origin xyz=0 0 0 rpy=0 0 0 -> xyz=0.0080046 -0.005 -0.055798 rpy=1.5708 -1.5708 0
- joint base_joint_gripper_left3: axis 1 0 0 -> 0 1 0; child gripper_left3 -> left_finger3; limit lower=-0.055 upper=-0.0027 effort=1.0 velocity=1.0 -> lower=0.01 upper=0.065 effort=0 velocity=0; origin xyz=0 0 0 rpy=0 0 0 -> xyz=0.0080046 -0.005 -0.055798 rpy=1.5708 -1.5708 0
- joint base_joint_gripper_right0: axis -1 0 0 -> 0 1 0; child gripper_right0 -> right_finger; limit lower=0.0027 upper=0.055 effort=1.0 velocity=1.0 -> lower=0.01 upper=0.065 effort=0 velocity=0; origin xyz=0 0 0 rpy=0 0 3.14159 -> xyz=-0.0081073 -0.007 -0.051048 rpy=1.5708 -1.5708 0
- joint base_joint_gripper_right1: axis -1 0 0 -> 0 1 0; child gripper_right1 -> right_finger1; limit lower=0.0027 upper=0.055 effort=1.0 velocity=1.0 -> lower=0.01 upper=0.065 effort=0 velocity=0; origin xyz=0 0 0 rpy=0 0 3.14159 -> xyz=-0.0081073 -0.007 -0.051048 rpy=1.5708 -1.5708 0
- joint base_joint_gripper_right2: axis -1 0 0 -> 0 1 0; child gripper_right2 -> right_finger2; limit lower=0.0027 upper=0.055 effort=1.0 velocity=1.0 -> lower=0.01 upper=0.065 effort=0 velocity=0; origin xyz=0 0 0 rpy=0 0 3.14159 -> xyz=-0.0081073 -0.007 -0.051048 rpy=1.5708 -1.5708 0
- joint base_joint_gripper_right3: axis -1 0 0 -> 0 1 0; child gripper_right3 -> right_finger3; limit lower=0.0027 upper=0.055 effort=1.0 velocity=1.0 -> lower=0.01 upper=0.065 effort=0 velocity=0; origin xyz=0 0 0 rpy=0 0 3.14159 -> xyz=-0.0081073 -0.007 -0.051048 rpy=1.5708 -1.5708 0
- joint tactile_sensor_joint_left3: parent finger_left3 -> left_finger3
- joint tactile_sensor_joint_right3: parent finger_right3 -> right_finger3

Commit message: fixed the prismatic direction of the GOAT joints

File: sim/pybullet/urdf_scalar_6DoF/urdf/SCALAR_6DoF_gripper_test.urdf (robot description, URDF)
Before this commit: robot SCALAR_6DoF, 62 links, 61 joints
Links:
- removed link tactile_sensor1
- removed link tactile_sensor2
Joints:
- removed joint tactile_sensor_joint_left3
- removed joint tactile_sensor_joint_right3
- joint base_joint_gripper_left0: limit lower=0.01 upper=0.065 effort=0 velocity=0 -> lower=-0.065 upper=-0.01 effort=0 velocity=0
- joint base_joint_gripper_left1: limit lower=0.01 upper=0.065 effort=0 velocity=0 -> lower=-0.065 upper=-0.01 effort=0 velocity=0
- joint base_joint_gripper_left2: limit lower=0.01 upper=0.065 effort=0 velocity=0 -> lower=-0.065 upper=-0.01 effort=0 velocity=0
- joint base_joint_gripper_left3: limit lower=0.01 upper=0.065 effort=0 velocity=0 -> lower=-0.065 upper=-0.01 effort=0 velocity=0
- joint fk_gripper0_joint: origin xyz=0.0 0 0.08 rpy=0 0 0 -> xyz=0.0 0 0.0 rpy=0 0 0
- joint fk_gripper1_joint: origin xyz=0.0 0 0.08 rpy=0 0 0 -> xyz=0.0 0 0.0 rpy=0 0 0
- joint fk_gripper2_joint: origin xyz=0.0 0 0.08 rpy=0 0 0 -> xyz=0.0 0 0.0 rpy=0 0 0
- joint fk_gripper3_joint: origin xyz=0.0 0 0.08 rpy=0 0 0 -> xyz=0.0 0 -0.048 rpy=0 0 0

Commit message: change orientation of holds so it works with new gripper, collision of gripper with obstacle still an issue and needs to be looked at

File: sim/pybullet/urdf_scalar_6DoF/urdf/SCALAR_6DoF_gripper_test.urdf (robot description, URDF)
Before this commit: robot SCALAR_6DoF, 60 links, 59 joints
Joints:
- joint fk_gripper0_joint: origin xyz=0.0 0 0.0 rpy=0 0 0 -> xyz=0.0 0 -0.048 rpy=0 0 0
- joint fk_gripper1_joint: origin xyz=0.0 0 0.0 rpy=0 0 0 -> xyz=0.0 0 -0.048 rpy=0 0 0
- joint fk_gripper2_joint: origin xyz=0.0 0 0.0 rpy=0 0 0 -> xyz=0.0 0 -0.048 rpy=0 0 0

File: sim/pybullet/urdf_scalar_6DoF/urdf/wall_camera_manyholds.urdf (robot description, URDF)
Before this commit: robot wall_with_hold, 9 links, 8 joints
Joints:
- joint wall_hold_joint: origin xyz=-0.12 0.32 0.07 rpy=3.14 0 0.0 -> xyz=-0.12 0.32 0.05 rpy=3.14 0 0.0
- joint wall_hold_joint2: origin xyz=0.12 0.42 0.07 rpy=3.14 0 0.0 -> xyz=0.12 0.42 0.05 rpy=3.14 0 0.0
- joint wall_hold_joint3: origin xyz=0.12 -0.32 0.07 rpy=3.14 0 0.0 -> xyz=0.12 -0.32 0.05 rpy=3.14 0 0.0
- joint wall_hold_joint4: origin xyz=-0.12 -0.32 0.07 rpy=3.14 0 0.0 -> xyz=-0.12 -0.32 0.05 rpy=3.14 0 0.0
- joint wall_hold_joint5: origin xyz=-0.12 0.5 0.07 rpy=3.14 0 0.0 -> xyz=-0.12 0.5 0.05 rpy=3.14 0 0.0
